Commit message: Rearranged sonar locations to align with N1-N16.  This is basically rotating all the sonars by 90 degrees.

File: fiducial_lib/loki.urdf (robot description, URDF)
Before this commit: robot loki, 17 links, 16 joints
Joints:
- joint base_sonar_1: origin xyz=0.088 0 0 rpy=0 0 0 -> xyz=-0.117 -0.055 0 rpy=0 0 -1.57
- joint base_sonar_10: origin xyz=-0.167813374 -0.021047589 0 rpy=0 0 -2.74889357 -> xyz=-0.138047589 0.050813374 0 rpy=0 0 1.96349541
- joint base_sonar_11: origin xyz=-0.155890873 -0.038890873 0 rpy=0 0 -2.35619449 -> xyz=-0.155890873 0.038890873 0 rpy=0 0 2.35619449
- joint base_sonar_12: origin xyz=-0.138047589 -0.050813374 0 rpy=0 0 -1.96349541 -> xyz=-0.167813374 0.021047589 0 rpy=0 0 2.74889357
- joint base_sonar_13: origin xyz=-0.117 -0.055 0 rpy=0 0 -1.57 -> xyz=-0.172 0 0 rpy=0 0 3.14159265
- joint base_sonar_14: origin xyz=0.0540476 -0.0508134 0 rpy=0 0 -1.17 -> xyz=-0.167813374 -0.021047589 0 rpy=0 0 -2.74889357
- joint base_sonar_15: origin xyz=0.0718909 -0.0388909 0 rpy=0 0 -0.79 -> xyz=-0.155890873 -0.038890873 0 rpy=0 0 -2.35619449
- joint base_sonar_16: origin xyz=0.0838134 -0.0210476 0 rpy=0 0 -0.39 -> xyz=-0.138047589 -0.050813374 0 rpy=0 0 -1.96349541
- joint base_sonar_2: origin xyz=0.0838134 0.0210476 0 rpy=0 0 0.39 -> xyz=0.0540476 -0.0508134 0 rpy=0 0 -1.17
- joint base_sonar_3: origin xyz=0.0718909 0.0388909 0 rpy=0 0 0.79 -> xyz=0.0718909 -0.0388909 0 rpy=0 0 -0.79
- joint base_sonar_4: origin xyz=0.0540476 0.0508134 0 rpy=0 0 1.17 -> xyz=0.0838134 -0.0210476 0 rpy=0 0 -0.39
- joint base_sonar_5: origin xyz=-0.117 0.055 0 rpy=0 0 1.57 -> xyz=0.088 0 0 rpy=0 0 0
- joint base_sonar_6: origin xyz=-0.138047589 0.050813374 0 rpy=0 0 1.96349541 -> xyz=0.0838134 0.0210476 0 rpy=0 0 0.39
- joint base_sonar_7: origin xyz=-0.155890873 0.038890873 0 rpy=0 0 2.35619449 -> xyz=0.0718909 0.0388909 0 rpy=0 0 0.79
- joint base_sonar_8: origin xyz=-0.167813374 0.021047589 0 rpy=0 0 2.74889357 -> xyz=0.0540476 0.0508134 0 rpy=0 0 1.17
- joint base_sonar_9: origin xyz=-0.172 0 0 rpy=0 0 3.14159265 -> xyz=-0.117 0.055 0 rpy=0 0 1.57

Commit message: Now label sonars starting from 0.

File: fiducial_lib/loki.urdf (robot description, URDF)
Before this commit: robot loki, 17 links, 16 joints
Links:
- removed link sonar_16
- added link sonar_0
Joints:
- removed joint base_sonar_16
- added joint base_sonar_0: type fixed, parent base_link, child sonar_0, origin xyz=-0.117 -0.055 0 rpy=0 0 -1.57
- joint base_sonar_1: origin xyz=-0.117 -0.055 0 rpy=0 0 -1.57 -> xyz=0.0540476 -0.0508134 0 rpy=0 0 -1.17
- joint base_sonar_10: origin xyz=-0.138047589 0.050813374 0 rpy=0 0 1.96349541 -> xyz=-0.155890873 0.038890873 0 rpy=0 0 2.35619449
- joint base_sonar_11: origin xyz=-0.155890873 0.038890873 0 rpy=0 0 2.35619449 -> xyz=-0.167813374 0.021047589 0 rpy=0 0 2.74889357
- joint base_sonar_12: origin xyz=-0.167813374 0.021047589 0 rpy=0 0 2.74889357 -> xyz=-0.172 0 0 rpy=0 0 3.14159265
- joint base_sonar_13: origin xyz=-0.172 0 0 rpy=0 0 3.14159265 -> xyz=-0.167813374 -0.021047589 0 rpy=0 0 -2.74889357
- joint base_sonar_14: origin xyz=-0.167813374 -0.021047589 0 rpy=0 0 -2.74889357 -> xyz=-0.155890873 -0.038890873 0 rpy=0 0 -2.35619449
- joint base_sonar_15: origin xyz=-0.155890873 -0.038890873 0 rpy=0 0 -2.35619449 -> xyz=-0.138047589 -0.050813374 0 rpy=0 0 -1.96349541
- joint base_sonar_2: origin xyz=0.0540476 -0.0508134 0 rpy=0 0 -1.17 -> xyz=0.0718909 -0.0388909 0 rpy=0 0 -0.79
- joint base_sonar_3: origin xyz=0.0718909 -0.0388909 0 rpy=0 0 -0.79 -> xyz=0.0838134 -0.0210476 0 rpy=0 0 -0.39
- joint base_sonar_4: origin xyz=0.0838134 -0.0210476 0 rpy=0 0 -0.39 -> xyz=0.088 0 0 rpy=0 0 0
- joint base_sonar_5: origin xyz=0.088 0 0 rpy=0 0 0 -> xyz=0.0838134 0.0210476 0 rpy=0 0 0.39
- joint base_sonar_6: origin xyz=0.0838134 0.0210476 0 rpy=0 0 0.39 -> xyz=0.0718909 0.0388909 0 rpy=0 0 0.79
- joint base_sonar_7: origin xyz=0.0718909 0.0388909 0 rpy=0 0 0.79 -> xyz=0.0540476 0.0508134 0 rpy=0 0 1.17
- joint base_sonar_8: origin xyz=0.0540476 0.0508134 0 rpy=0 0 1.17 -> xyz=-0.117 0.055 0 rpy=0 0 1.57
- joint base_sonar_9: origin xyz=-0.117 0.055 0 rpy=0 0 1.57 -> xyz=-0.138047589 0.050813374 0 rpy=0 0 1.96349541
